Commit message: Fine adjustment of contents

File: urdf/gripper/gripper.gazebo.xacro (robot description, xacro)
@@ -22,6 +22,6 @@
     </gazebo>
     <gazebo reference="prismatic_finger_${name}">
-      <!-- <provideFeedback>true</provideFeedback> -->
-      <!-- <implicitSpringDamper>true</implicitSpringDamper> -->
+      <provideFeedback>true</provideFeedback>
+      <implicitSpringDamper>true</implicitSpringDamper>
     </gazebo>
   </xacro:macro>

File: urdf/gripper/gripper.transmission.xacro (robot description, xacro)
@@ -7,5 +7,5 @@
 	<!-- <hardwareInterface>hardware_interface/PositionJointInterface</hardwareInterface> -->
 	<hardwareInterface>hardware_interface/VelocityJointInterface</hardwareInterface>
-	<!-- <hardwareInterface>EffortJointInterface</hardwareInterface> -->
+	<!-- <hardwareInterface>hardware_interface/EffortJointInterface</hardwareInterface> -->
       </joint>
       <actuator name="prismatic_finger_${name}_motor">
@@ -13,5 +13,5 @@
 	<!-- <hardwareInterface>hardware_interface/PositionJointInterface</hardwareInterface> -->
 	<hardwareInterface>hardware_interface/VelocityJointInterface</hardwareInterface>
-	<!-- <hardwareInterface>EffortJointInterface</hardwareInterface> -->
+	<!-- <hardwareInterface>hardware_interface/EffortJointInterface</hardwareInterface> -->
       </actuator>
     </transmission>

File: urdf/gripper/gripper.urdf.xacro (robot description, xacro)
@@ -54,9 +54,4 @@
         <xacro:insert_block name="root_origin"/>
 	<mass value="0.002" />
-      <!-- 	<inertia -->
-      <!--       ixx="1.0" ixy="1.0" ixz="1.0" -->
-      <!--       iyy="1.0" iyz="1.0" -->
-      <!--       izz="1.0" /> -->
-      <!-- </inertial> -->
       	<inertia
             ixx="3.30140945222581E-06" ixy="6.88214269644119E-22" ixz="1.69538938348869E-20"

File: urdf/mobile_base/mobile_base.urdf.xacro (robot description, xacro)
@@ -86,10 +86,4 @@
 	</geometry>
       </visual>
-      <!-- <collision> -->
-      <!-- 	<origin rpy="0 0 0" xyz="0 0 0"/> -->
-      <!-- 	<geometry> -->
-      <!-- 	  <box size=".001 .001 .001" /> -->
-      <!-- 	</geometry> -->
-      <!-- </collision> -->
     </link>
     <link name="${name}_caster">
@@ -108,10 +102,4 @@
 		                                         izz="0.01248008322"/>
       </inertial>
-      <!-- <collision> -->
-      <!-- 	<origin rpy="${PI} 0 0" xyz="0 0 0"/> -->
-      <!-- 	<geometry> -->
-      <!-- 	  <mesh filename="package://rls_robot_description/meshes/stl/caster.stl"/> -->
-      <!-- 	</geometry> -->
-      <!-- </collision> -->
     </link>
     <link name="${name}_small_wheel">
@@ -186,5 +174,4 @@
   </joint>
   <xacro:macro name="small_wheel_joint" params="name *origin">
-    <!-- <joint name="${name}_bearing_joint" type="fixed"> -->
     <joint name="${name}_bearing_joint" type="prismatic">
       <parent link="base_link"/>

File: urdf/symmarm/symmarm.transmission.xacro (robot description, xacro)
@@ -6,9 +6,9 @@
     <joint name="joint${name}">
       <hardwareInterface>hardware_interface/VelocityJointInterface</hardwareInterface>
-      <!-- <hardwareInterface>EffortJointInterface</hardwareInterface> -->
+      <!-- <hardwareInterface>hardware_interface/EffortJointInterface</hardwareInterface> -->
     </joint>
     <actuator name="joint${name}_motor">
       <hardwareInterface>hardware_interface/VelocityJointInterface</hardwareInterface>
-      <!-- <hardwareInterface>EffortJointInterface</hardwareInterface> -->
+      <!-- <hardwareInterface>hardware_interface/EffortJointInterface</hardwareInterface> -->
       <mechanicalReduction>${reduction}</mechanicalReduction>
     </actuator>
